File: radio.kicad_sch (KiCad schematic)
At the start: 14 parts, among them U4 MCP6002-xMS

Commit message: refactor hierarchical sheets to use sheet pins
Changed lines of the file:
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@@
+	)
+	(junction
+		(at 208.28 101.6)
+		(diameter 0)
+		(color 0 0 0 0)
 	)
 	(junction
@@
 	(wire
 		(pts
-			(xy 196.85 101.6) (xy 213.36 101.6)
+			(xy 196.85 101.6) (xy 208.28 101.6)
 		)
 		(stroke
@@
 	(wire
 		(pts
+			(xy 208.28 101.6) (xy 213.36 101.6)
+		)
+		(stroke
+			(width 0)
+			(type default)
+		)
+	)
+	(wire
+		(pts
 			(xy 69.85 50.8) (xy 69.85 53.34)
 		)
@@
 		(pts
 			(xy 69.85 60.96) (xy 69.85 63.5)
+		)
+		(stroke
+			(width 0)
+			(type default)
+		)
+	)
+	(wire
+		(pts
+			(xy 213.36 96.52) (xy 208.28 96.52)
+		)
+		(stroke
+			(width 0)
+			(type default)
+		)
+	)
+	(wire
+		(pts
+			(xy 208.28 96.52) (xy 208.28 101.6)
 		)
 		(stroke
@@
 		)
 	)
+	(hierarchical_label "antenna_sig_out"
+		(shape output)
+		(at 213.36 96.52 0)
+		(effects
+			(font
+				(size 1.27 1.27)
+			)
+			(justify left)
+		)
+	)

Commit message: WIP relayout of board
Parts:
- removed AE1: Antenna, symbol Device:Antenna
- added AE1: ~, antenna:capacitive_coupled_50mmx8mm, symbol antenna:capacitive_pickup_50mmx8mm
- C10, C11, C8, C9: footprint Capacitor_SMD:C_0603_1608Metric -> Capacitor_SMD:C_0402_1005Metric
- R18, R19, R20, R21, R22, R23, R24: footprint Resistor_SMD:R_0603_1608Metric -> Resistor_SMD:R_0402_1005Metric
Connections:
- net GND: now also AE1.2 (GND)
- net at R20.2, R21.2: now also AE1.1 (Signal)
- net cc_antenna_out renamed antenna_sig_out

Commit message: Board V3
Parts:
- removed C8: 0.1uF, Capacitor_SMD:C_0402_1005Metric, symbol Device:C
- removed R18, R19: 100k, Resistor_SMD:R_0402_1005Metric, symbol Device:R
- AE1: now left out of the parts list
- C10: Est Cost (1000) (none) -> 0.0016; LCSC (none) -> https://www.lcsc.com/product-detail/C6119800.html; Manufacturer (none) -> HRE; Part No (none) -> CGA0402X7R224K160GT; Type (none) -> SMD; Vendor https://www.lcsc.com/product-detail/C519556.html -> (none)
- C11: value 0.1uF -> 100nF; Est Cost 0.002 -> (none); Est Cost (1000) (none) -> 0.0007; LCSC (none) -> https://www.lcsc.com/product-detail/C22435938.html; Manufacturer (none) -> HRE; Part No (none) -> CGA0402X7R104K6R3GT; Type (none) -> SMD; Vendor https://www.lcsc.com/product-detail/C6119883.html -> (none)
- C9: Est Cost 0.0032 -> (none); Est Cost (1000) (none) -> 0.0007; LCSC (none) -> https://www.lcsc.com/product-detail/C22435961.html; Manufacturer (none) -> HRE; Part No (none) -> CGA0402X7R821K500GT; Type (none) -> SMD; Vendor https://www.lcsc.com/product-detail/C107057.html -> (none)
- D3: Est Cost 0.0056 -> (none); Est Cost (1000) (none) -> 0.0063; Height (none) -> 1.1mm; LCSC (none) -> https://www.lcsc.com/product-detail/C909763.html?s_z=n_BAV99; Manufacturer (none) -> GOODWORK; Part No (none) -> BAV99; Type (none) -> SMD; Vendor https://www.lcsc.com/product-detail/C909763.html?s_z=n_BAV99 -> (none)
- R20: Est Cost 0.0006 -> (none); Est Cost (1000) (none) -> 0.0004; LCSC (none) -> https://www.lcsc.com/product-detail/C2906900.html; Manufacturer (none) -> FOJAN; Part No (none) -> FRC0402J105 TS; Type (none) -> SMD; Vendor https://www.lcsc.com/product-detail/C49254192.html -> (none)
- R21: Est Cost 0.0006 -> (none); Est Cost (1000) (none) -> 0.0004; LCSC (none) -> https://www.lcsc.com/product-detail/C2906941.html; Manufacturer (none) -> FOJAN; Part No (none) -> FRC0402J472 TS; Type (none) -> SMD; Vendor https://www.lcsc.com/product-detail/C49254210.html -> (none)
- R22, R23: Est Cost 0.0007 -> (none); Est Cost (1000) (none) -> 0.0003; LCSC (none) -> https://www.lcsc.com/product-detail/C3017479.html; Manufacturer (none) -> VO; Part No (none) -> SCR0402J1K; Type (none) -> SMD; Vendor https://www.lcsc.com/product-detail/C2907002.html -> (none)
- R24: Est Cost 0.0053 -> (none); Est Cost (1000) (none) -> 0.0004; LCSC (none) -> https://www.lcsc.com/product-detail/C2998093.html; Manufacturer (none) -> FOJAN; Part No (none) -> FRC0402F4021TS; Type (none) -> SMD; Vendor https://www.lcsc.com/product-detail/C2984443.html -> (none)
- U4: footprint Package_TO_SOT_SMD:SuperSOT-8 -> Package_SO:SOP-8_3.76x4.96mm_P1.27mm; Est Cost 0.048 -> (none); Est Cost (1000) (none) -> 0.048; Height (none) -> 1.8mm; LCSC (none) -> https://www.lcsc.com/product-detail/C48997707.html?s_z=n_MC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; Manufacturer (none) -> lingxingic; Part No (none) -> MCP6002T-I/SN(LX); Type (none) -> SMD; Vendor https://www.lcsc.com/product-detail/C48997707.html?s_z=n_MC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 -> (none)
Connections:
- net 1V6: now reaches R20.1
Other:
- moved on the sheet: R20
